File: payload1_board/payload1_board.kicad_sch (KiCad schematic)
At the start: 0 parts

Commit message: Add SAMD21 schematic
Other:
- added sheet MCU (mcu.kicad_sch)
Changed lines of the file:
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@@
 	(generator_version "9.0")
 	(paper "A4")
+	(sheet
+		(at 22.86 25.4)
+		(size 63.5 39.37)
+		(exclude_from_sim no)
+		(in_bom yes)
+		(on_board yes)
+		(dnp no)
+		(fields_autoplaced yes)
+		(stroke
+			(width 0.1524)
+			(type solid)
+		)
+		(fill
+			(color 0 0 0 0.0000)
+		)
+		(property "Sheetname" "MCU"
+			(at 22.86 24.6884 0)
+			(effects
+				(font
+					(size 1.27 1.27)
+				)
+				(justify left bottom)
+			)
+		)
+		(property "Sheetfile" "mcu.kicad_sch"
+			(at 22.86 65.3546 0)
+			(effects
+				(font
+					(size 1.27 1.27)
+				)
+				(justify left top)
+			)
+		)
+		(instances
+			(project "payload1_board"
+				(path "/e2d2dcec-a18d-4e9a-9957-29b22748b89d"
+					(page "2")
+				)
+			)
+		)
+	)
 	(sheet_instances
 		(path "/"

Commit message: Update schematic
Other:
- added sheet GPS (gps.kicad_sch)
- added sheet RF (rf.kicad_sch)
Changed lines of the file:
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@@
 	(paper "A4")
 	(sheet
-		(at 22.86 25.4)
-		(size 63.5 39.37)
+		(at 135.89 31.75)
+		(size 34.29 21.59)
+		(exclude_from_sim no)
+		(in_bom yes)
+		(on_board yes)
+		(dnp no)
+		(fields_autoplaced yes)
+		(stroke
+			(width 0.1524)
+			(type solid)
+		)
+		(fill
+			(color 0 0 0 0.0000)
+		)
+		(property "Sheetname" "GPS"
+			(at 135.89 31.0384 0)
+			(effects
+				(font
+					(size 1.27 1.27)
+				)
+				(justify left bottom)
+			)
+		)
+		(property "Sheetfile" "gps.kicad_sch"
+			(at 135.89 53.9246 0)
+			(effects
+				(font
+					(size 1.27 1.27)
+				)
+				(justify left top)
+			)
+		)
+		(instances
+			(project "payload1_board"
+				(path "/ea597178-b44d-4db9-826c-8f86e8d231f0"
+					(page "4")
+				)
+			)
+		)
+	)
+	(sheet
+		(at 30.48 31.75)
+		(size 40.64 21.59)
 		(exclude_from_sim no)
 		(in_bom yes)
@@
 		)
 		(property "Sheetname" "MCU"
-			(at 22.86 24.6884 0)
+			(at 30.48 31.0384 0)
 			(effects
 				(font
@@
 		)
 		(property "Sheetfile" "mcu.kicad_sch"
-			(at 22.86 65.3546 0)
+			(at 30.48 53.9246 0)
 			(effects
 				(font
@@
 		(instances
 			(project "payload1_board"
-				(path "/e2d2dcec-a18d-4e9a-9957-29b22748b89d"
+				(path "/ea597178-b44d-4db9-826c-8f86e8d231f0"
 					(page "2")
 				)
 			)
+		)
+	)
+	(sheet
+		(at 81.28 31.75)
+		(size 41.91 21.59)
+		(exclude_from_sim no)
+		(in_bom yes)
+		(on_board yes)
+		(dnp no)
+		(fields_autoplaced yes)
+		(stroke
+			(width 0.1524)
+			(type solid)
+		)
+		(fill
+			(color 0 0 0 0.0000)
+		)
+		(property "Sheetname" "RF"
+			(at 81.28 31.0384 0)
+			(effects
+				(font
+					(size 1.27 1.27)
+				)
+				(justify left bottom)
+			)
+		)
+		(property "Sheetfile" "rf.kicad_sch"
+			(at 81.28 53.9246 0)
+			(effects
+				(font
+					(size 1.27 1.27)
+				)
+				(justify left top)
+			)
+		)
+		(instances
+			(project "payload1_board"
+				(path "/ea597178-b44d-4db9-826c-8f86e8d231f0"
+					(page "3")
+				)
+			)
