File: payload1_board/payload1_board.kicad_sch (KiCad schematic)
At the start: 0 parts

Commit message: update
Other:
- company: Sanie Peralta, Alejandro Campo -> Introduccion a la ingenieria satelital
- title: Payload 2nd stage -> Payload 2nd PCB
Changed lines of the file:
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@@
 	(paper "A4")
 	(title_block
-		(title "Payload 2nd stage")
+		(title "Payload 2nd PCB")
 		(date "01/04/2026")
-		(company "Sanie Peralta, Alejandro Campo")
+		(company "Introduccion a la ingenieria satelital")
+		(comment 1 "Sanie Peralta, Alejandro Campo")
 	)
 	(sheet
