File: payload1_board/mcu.kicad_sch (KiCad schematic)
At the start: 26 parts, among them IC1 STM32F411CEU7, J1 Screw_Terminal_01x04, J3 Screw_Terminal_01x02, SW1 SW_SPST, SW2 SW_SPST, SW3 SW_SPST, Y2 16MHz

Commit message: update
Other:
- company: (none) -> Introduccion a la ingenieria satelital
- title: (none) -> Payload 2nd PCB
Changed lines of the file:
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@@
 	(generator_version "9.0")
 	(paper "A4")
+	(title_block
+		(title "Payload 2nd PCB")
+		(company "Introduccion a la ingenieria satelital")
+		(comment 1 "Sanie Peralta, Alejandro Campo")
+	)
 	(text "User KEY"
 		(exclude_from_sim no)
