File: payload1_board/ocp.kicad_sch (KiCad schematic)
At the start: 12 parts, among them Q1 DTC114E, Q2 SSM6K403TU_LF, Q3 DTC114E, U1 LTC4361HTS8-2-TRMPBF

Commit message: update
Other:
- company: (none) -> Introduccion a la ingenieria satelital
- title: (none) -> Payload 2nd PCB
Changed lines of the file:
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@@
 	(generator_version "9.0")
 	(paper "A4")
+	(title_block
+		(title "Payload 2nd PCB")
+		(company "Introduccion a la ingenieria satelital")
+		(comment 1 "Sanie Peralta, Alejandro Campo")
+	)
 	(junction
 		(at 242.062 86.106)
