File: payload1_board/sensores.kicad_sch (KiCad schematic)
At the start: 10 parts, among them U3 AIS328DQTR, U4 MMC5983MA, U5 I3G4250DTR

Commit message: sensors done
Parts:
- added C44: 100nf, symbol Device:C
- added C45: 10uf, symbol Device:C
- added R6, R7: 10k, symbol Device:R
Connections:
- net GND: now also U5.8 (RES), C44.2, C45.2
- net OCP_TO_GYRO: now reaches U5.1 (VDD_IO)
- net OCP_TO_GYRO: now also U5.15 (RES), U5.16 (VDD), C44.1, C45.1, R7.1
- net IMU_SCL_TO_STM_SCK: now reaches U5.2 (SCL/SPC)
- net IMU_SCL_TO_STM_SCK: now also U3.11 (SPC/SCL), U4.1 (SCL/SPI_SCK)
- net IMU_SDI_TO_STM_MOSI: now reaches U5.3 (SDA/SDI/SDO)
- net IMU_SDI_TO_STM_MOSI: now also U3.16 (SDI/SDO/SDA), U4.16 (SDA/SPI_SDI)
- net IMU_SDO_TO_STM_MISO: now reaches U5.4 (SDO/SA0)
- net IMU_SDO_TO_STM_MISO: now also U3.15 (SDO/SA0), U4.5 (SPI_SDO)
- net GYRO_CS_TO_STM_NSS: now reaches U5.5 (CS)
- net GYRO_CS_TO_STM_NSS: now also R7.2
- net GYRO_INT2_TO_STM: now reaches U5.6 (DRDY/INT2)
- net GYRO_INT1_TO_STM: now reaches U5.7 (INT1)
- net OCP_TO_ACCEL: now reaches C38.1, C39.1, U3.5 (VDD)
- net OCP_TO_ACCEL: now also U3.14 (VDD_IO), R6.1
- net ACCEL_CS_TO_STM_NSS: now reaches U3.12 (CS)
- net ACCEL_CS_TO_STM_NSS: now also R6.2
- net ACCEL_INT2_TO_STM: now reaches U3.3 (INT_2)
- net ACCEL_INT1_TO_STM: now reaches U3.7 (INT_1)
- net OCP_TO_MAG: now reaches C43.2, U4.2 (VDD)
- net OCP_TO_MAG: now also U4.13 (VDDIO)
- net MAG_INT_TO_STM: now reaches U4.15 (INT)
- net MAG_CS_TO_STM_NSS: now reaches U4.4 (SPI_CS)
Other:
- moved on the sheet: C40, C41, C42, C43, R2, U4, U5

Commit message: 1st debugging
Other:
- note added: "ACCEL"
- note added: "GYRO"
- note added: "MAG"
