File: payload1_board/sensores.kicad_sch (KiCad schematic)
At the start: 14 parts, among them U2 AIS328DQTR, U3 MMC5983MA, U4 I3G4250DTR

Commit message: update
Other:
- company: (none) -> Introduccion a la ingenieria satelital
- title: (none) -> Payload 2nd PCB
Changed lines of the file:
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@@
 	(generator_version "9.0")
 	(paper "A4")
+	(title_block
+		(title "Payload 2nd PCB")
+		(company "Introduccion a la ingenieria satelital")
+		(comment 1 "Sanie Peralta, Alejandro Campo")
+	)
 	(text "ACCEL\n"
 		(exclude_from_sim no)
