File: payload1_board/io_conn.kicad_sch (KiCad schematic)
At the start: 8 parts, among them J2 USB_B_Micro, J4 Screw_Terminal_01x03, U5 ADP122AUJZ-3.3-R7

Commit message: update
Other:
- company: (none) -> Introduccion a la ingenieria satelital
- title: (none) -> Payload 2nd PCB
Changed lines of the file:
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@@
 	(generator_version "9.0")
 	(paper "A4")
+	(title_block
+		(title "Payload 2nd PCB")
+		(company "Introduccion a la ingenieria satelital")
+		(comment 1 "Sanie Peralta, Alejandro campo")
+	)
 	(text "USB\n"
 		(exclude_from_sim no)
